Commit message: Change arm_base_link location to be on table (not on turtlebot)

File: turtlebot_arm_description/urdf/pincher_arm.urdf.xacro (robot description, xacro)
@@ -22,5 +22,7 @@
       <!-- Place the "floating" arm at the location it should be if mounted on a turtlebot,
            as pick and place and other demos assume this location -->
-      <origin xyz="0.1 0.03 0.435"/>
+      <!-- origin xyz="0.1 0.03 0.435"/-->
+	<!-- Here changed to assume that arm is mounted on the table -->
+	<origin xyz="-0.0249 0.0 0.0634" />
     </turtlebot_arm>
 </robot>

Commit message: another urdf fix, to center of servo

File: turtlebot_arm_description/urdf/pincher_arm.urdf.xacro (robot description, xacro)
@@ -24,5 +24,5 @@
       <!-- origin xyz="0.1 0.03 0.435"/-->
 	<!-- Here changed to assume that arm is mounted on the table -->
-	<origin xyz="-0.0249 0.0 0.0634" />
+	<origin xyz="-0.0444 0.0 0.0634" />
     </turtlebot_arm>
 </robot>
