Commit message: rail rotation done

File: turtlebot_arm_description/urdf/arm_hardware.xacro (robot description, xacro)
@@ -270,5 +270,5 @@
       <xacro:box_inertia length="0.002" width="0.040" height="0.075" mass="0.00001"/>
       <visual>
-        <origin xyz="0.016 0 -.015 " rpy="${M_PI} ${-M_PI/2} ${M_PI/2}"/>
+        <origin xyz="0.016 0 -.015 " rpy="${M_PI/2} ${M_PI/2} ${M_PI/2}"/>
         <geometry>
           <mesh filename="package://turtlebot_arm_description/meshes/pincher_finger_base.stl" scale=".01 .01 .01"/>

Commit message: Rail changed + servo rotated + grip2 mimic joint

File: turtlebot_arm_description/urdf/arm_hardware.xacro (robot description, xacro)
@@ -268,7 +268,7 @@
     </joint>
     <link name="${name}_link">
-      <xacro:box_inertia length="0.002" width="0.040" height="0.075" mass="0.00001"/>
-      <visual>
-        <origin xyz="0.016 0 -.015 " rpy="${M_PI/2} ${M_PI/2} ${M_PI/2}"/>
+      <xacro:box_inertia length="0.002" width="0.065" height="0.075" mass="0.00001"/>
+      <visual>
+        <origin xyz="0.016 0 -.015 " rpy="0 0 0"/>
         <geometry>
           <mesh filename="package://turtlebot_arm_description/meshes/pincher_finger_base.stl" scale=".01 .01 .01"/>
@@ -279,5 +279,5 @@
         <origin xyz="0.016 0.0 -0.015" rpy="0 0 0"/>
         <geometry>
-          <box size="0.002 0.040 0.075"/>
+          <box size="0.002 0.065 0.075"/>
         </geometry>
       </collision>

File: turtlebot_arm_description/urdf/pincher_gripper.xacro (robot description, xacro)
@@ -7,39 +7,43 @@
     <!-- gripper joint -->
     <dynamixel_AX12_fixed parent="arm_wrist_F3_0_link" name="gripper_servo" >
-      <origin xyz="0 0 ${-AX12_WIDTH/2}" rpy="${M_PI/2} ${M_PI} ${M_PI/2}"/>
+      <origin xyz="0 0 ${-AX12_WIDTH/2}" rpy="${M_PI/2} 0 ${M_PI/2}"/>
     </dynamixel_AX12_fixed>
      <gripper_finger_base parent="gripper_servo_link" name="gripper_finger_base" color="${color}">
-      <origin xyz="0.01  ${AX12_WIDTH} 0" rpy="${M_PI/2} ${-M_PI} ${M_PI/2}"/>
+      <origin xyz="${-(0.065-AX12_HEIGHT)} ${-AX12_WIDTH} ${-AX12_LENGTH/2}" rpy="${M_PI/2} 0 0"/>
     </gripper_finger_base>
      <!-- Finger 1 -->
     <joint name="gripper_joint" type="prismatic">
-      <origin xyz="0 0 0" rpy="0 0 0"/>
+      <origin xyz="0 0 0" rpy="0 0 ${-M_PI/2}"/>
       <axis xyz="1 0 0"/>
       <limit effort="30" velocity="0.5" lower="0.002" upper="0.031"/>
-      <parent link="gripper_servo_link"/>
+      <parent link="gripper_finger_base_link"/>
       <child link="gripper_active_link"/>
     </joint>
     <pincher_gripper name="gripper_active" color="${color}" >
-      <origin xyz="-0.0086 0.0414 0" rpy="${-M_PI/2} 0 0"/>
+<!--      <origin xyz="-0.0086 0.0414 0" rpy="${-M_PI/2} 0 0"/>-->
+	<origin xyz="${-0.0086+AX12_LENGTH/3} ${0.0414-AX12_HEIGHT/3} 0" rpy="0 0 0"/>
     </pincher_gripper>
     <!-- Finger 2 -->
-    <!-- Note: currently static but should be a Mimic of Finger 1 -->
+    <!-- Note: currently static but should be a Mimic of Finger 1
     <joint name="gripper2_joint" type="fixed">
-      <parent link="gripper_servo_link"/>
+      <origin xyz="0 0 0" rpy="0 0 ${-M_PI/2}"/>
+      <parent link="gripper_finger_base_link"/>
       <child link="gripper_active2_link"/>
-    </joint>
+    </joint-->
     <pincher_gripper name="gripper_active2" color="${color}" >
-      <origin xyz="-0.0314 0.0414 0" rpy="${-M_PI/2} ${M_PI} 0"/>
+<!--      <origin xyz="-0.0314 0.0414 0" rpy="${-M_PI/2} ${M_PI} 0"/>-->
+	<origin xyz="${-0.0314+AX12_LENGTH/3} ${0.0414-AX12_HEIGHT/3} 0" rpy="${M_PI} ${M_PI} 0"/>
     </pincher_gripper>
     <!-- Using Mimic -->
     <!-- gripper 2 joint -->
-    <!--  ### Mimic would be better but causes Missing Joint error in Moveit
+    <!--  ### Mimic would be better but causes Missing Joint error in Moveit -->
       <joint name="gripper2_joint" type="prismatic">
-      <origin xyz="0 0 0" rpy="0 0 0"/>
-      <axis xyz="0 0 1"/>
+<!--      <origin xyz="0 0 0" rpy="0 0 0"/> -->
+      <origin xyz="0 0 0" rpy="0 0 ${-M_PI/2}"/>
+      <axis xyz="1 0 0"/>
       <limit effort="30" velocity="0.5" lower="0.002" upper="0.031"/>
-      <parent link="gripper_servo_link"/>
+      <parent link="gripper_finger_base_link"/>
       <child link="gripper_active2_link"/>
       <mimic joint="gripper_joint" multiplier="-.5"  offset = "0"/>
-    </joint-->
+    </joint>
 </robot>

Commit message: Camera base added + gripper rail height fixed

File: turtlebot_arm_description/urdf/arm_hardware.xacro (robot description, xacro)
@@ -312,3 +312,26 @@
     </gazebo>
   </xacro:macro>
+    <xacro:macro name="camera_base" params="name color *origin">
+      <link name="${name}_link">
+      <xacro:box_inertia length="0.033" width="0.039" height="0.049" mass="0.00001"/>
+      <visual>
+        <xacro:insert_block name="origin"/>
+        <geometry>
+          <mesh filename="package://turtlebot_arm_description/meshes/camera_base.stl" scale=".01 .01 .01"/>
+        </geometry>
+        <material name="${color}"/>
+      </visual>
+      <collision>
+        <xacro:insert_block name="origin"/>
+        <geometry>
+          <box size="0.033 0.039 0.049"/>
+        </geometry>
+      </collision>
+    </link>
+    <gazebo reference="${name}_link">
+      <material>Gazebo/${color}</material>
+      <selfCollide>true</selfCollide>
+      <gravity>true</gravity>
+    </gazebo>
+  </xacro:macro>
 </robot>

File: turtlebot_arm_description/urdf/pincher_gripper.xacro (robot description, xacro)
@@ -10,5 +10,5 @@
     </dynamixel_AX12_fixed>
      <gripper_finger_base parent="gripper_servo_link" name="gripper_finger_base" color="${color}">
-      <origin xyz="${-(0.065-AX12_HEIGHT)} ${-AX12_WIDTH} ${-AX12_LENGTH/2}" rpy="${M_PI/2} 0 0"/>
+      <origin xyz="${-(0.065-AX12_HEIGHT)} ${-AX12_WIDTH+0.004} ${-AX12_LENGTH/2}" rpy="${M_PI/2} 0 0"/>
     </gripper_finger_base>
      <!-- Finger 1 -->
@@ -22,22 +22,21 @@
     <pincher_gripper name="gripper_active" color="${color}" >
 <!--      <origin xyz="-0.0086 0.0414 0" rpy="${-M_PI/2} 0 0"/>-->
-	<origin xyz="${-0.0086+AX12_LENGTH/3} ${0.0414-AX12_HEIGHT/3} 0" rpy="0 0 0"/>
+	<origin xyz="${-0.0086+AX12_LENGTH/3} ${0.0414-AX12_HEIGHT/3} 0.005" rpy="0 0 0"/>
     </pincher_gripper>
     <!-- Finger 2 -->
-    <!-- Note: currently static but should be a Mimic of Finger 1
+    <!-- Note: currently static but should be a Mimic of Finger 1 -->
     <joint name="gripper2_joint" type="fixed">
       <origin xyz="0 0 0" rpy="0 0 ${-M_PI/2}"/>
       <parent link="gripper_finger_base_link"/>
       <child link="gripper_active2_link"/>
-    </joint-->
+    </joint>
     <pincher_gripper name="gripper_active2" color="${color}" >
 <!--      <origin xyz="-0.0314 0.0414 0" rpy="${-M_PI/2} ${M_PI} 0"/>-->
-	<origin xyz="${-0.0314+AX12_LENGTH/3} ${0.0414-AX12_HEIGHT/3} 0" rpy="${M_PI} ${M_PI} 0"/>
+	<origin xyz="${-0.0314+AX12_LENGTH/3} ${0.0414-AX12_HEIGHT/3} 0.005" rpy="${M_PI} ${M_PI} 0"/>
     </pincher_gripper>
     <!-- Using Mimic -->
     <!-- gripper 2 joint -->
-    <!--  ### Mimic would be better but causes Missing Joint error in Moveit -->
+    <!--  ### Mimic would be better but causes Missing Joint error in Moveit
       <joint name="gripper2_joint" type="prismatic">
-<!--      <origin xyz="0 0 0" rpy="0 0 0"/> -->
       <origin xyz="0 0 0" rpy="0 0 ${-M_PI/2}"/>
       <axis xyz="1 0 0"/>
@@ -46,4 +45,13 @@
       <child link="gripper_active2_link"/>
       <mimic joint="gripper_joint" multiplier="-.5"  offset = "0"/>
+    </joint>  -->
+     <!-- Camera adapter -->
+    <joint name="camera_base_joint" type="fixed">
+      <origin xyz="-0.0177 0.0192 -0.039" rpy="0 0 0"/>
+      <parent link="gripper_finger_base_link"/>
+      <child link="camera_base_link"/>
     </joint>
+    <camera_base name="camera_base" color="${color}" >
+	<origin xyz="0 0 0" rpy="0 0 0"/>
+    </camera_base>
 </robot>

Commit message: Robot description added - collision fixed and gripper closed fixed

File: turtlebot_arm_description/urdf/arm_hardware.xacro (robot description, xacro)
@@ -277,5 +277,5 @@
       </visual>
       <collision>
-        <origin xyz="0.016 0.0 -0.015" rpy="0 0 0"/>
+        <origin xyz="0.016 0.0 -0.015" rpy="0 ${M_PI/2} 0"/>
         <geometry>
           <box size="0.002 0.065 0.075"/>
@@ -325,5 +325,5 @@
         <xacro:insert_block name="origin"/>
         <geometry>
-          <box size="0.033 0.039 0.049"/>
+          <box size="0.039 0.032 0.049"/>
         </geometry>
       </collision>
