Commit message: Added camera to arm + arm to turtlebot3

File: turtlebot_arm_description/urdf/pincher_arm.urdf (robot description, URDF)
Before this commit: robot turtlebot_arm, 24 links, 23 joints
Links:
- added link camera_base_link, mass 1e-05; collision box size=0.033 0.039 0.049; visual mesh filename=package://turtlebot_arm_description/meshes/camera_base.stl scale=.01 .01 .01
- link gripper_active2_link: geometry collision box size=0.023 0.028 0.038; visual mesh filename=package://turtlebot_arm_description/meshes/pincher_finger.s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 scale=.01 .01 .01
- link gripper_active_link: geometry collision box size=0.023 0.028 0.038; visual mesh filename=package://turtlebot_arm_description/meshes/pincher_finger.s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 scale=.01 .01 .01
- link gripper_finger_base_link: geometry collision box size=0.002 0.065 0.075; visual mesh filename=package://turtlebot_arm_description/meshes/pincher_finger_b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 scale=.01 .01 .01
Joints:
- added joint camera_base_joint: type fixed, parent gripper_finger_base_link, child camera_base_link, origin xyz=-0.0177 0.0192 -0.039 rpy=0 0 0
- joint arm_base_joint: origin xyz=0.1 0.03 0.435 -> xyz=-0.0444 0.0 0.0634
- joint gripper2_joint: origin (none) -> xyz=0 0 0 rpy=0 0 -1.570795; parent gripper_servo_link -> gripper_finger_base_link
- joint gripper_finger_base_joint: origin xyz=0.01  0.038 0 rpy=1.570795 -3.14159 1.570795 -> xyz=-0.0265 -0.034 -0.025 rpy=1.570795 0 0
- joint gripper_joint: origin xyz=0 0 0 rpy=0 0 0 -> xyz=0 0 0 rpy=0 0 -1.570795; parent gripper_servo_link -> gripper_finger_base_link
- joint gripper_servo_joint: origin xyz=0 0 -0.019 rpy=1.570795 3.14159 1.570795 -> xyz=0 0 -0.019 rpy=1.570795 0 1.570795

File: turtlebot_arm_description/urdf/pincher_arm.urdf.xacro (robot description, xacro)
@@ -16,13 +16,14 @@
      <!-- Pincher arm is same as Turtlebot -->
     <xacro:include filename="$(find turtlebot_arm_description)/urdf/turtlebot_arm.xacro"/>
+<!-- Connected to turtlebot3 -->
     <!-- As we don't have here a turtlebot base, add a base_link link as its location reference -->
-    <link name="base_link"/>
+<!--   <link name="base_link"/> -->
     <!-- Turtlebot arm macro -->
-    <turtlebot_arm parent="base_link" color="Gray" gripper_color="Gray"   pincher_gripper="true" turtlebot_gripper="false">
+<!--    <turtlebot_arm parent="base_link" color="Gray" gripper_color="Gray"   pincher_gripper="true" turtlebot_gripper="false"> -->
       <!-- Place the "floating" arm at the location it should be if mounted on a turtlebot,
            as pick and place and other demos assume this location -->
       <!-- origin xyz="0.1 0.03 0.435"/-->
 	<!-- Here changed to assume that arm is mounted on the table -->
-	<origin xyz="-0.0444 0.0 0.0634" />
-    </turtlebot_arm>
+<!--	<origin xyz="-0.0444 0.0 0.0634" />
+    </turtlebot_arm> -->
 </robot>

File: turtlebot_arm_description/urdf/pincher_gripper.xacro (robot description, xacro)
@@ -10,5 +10,5 @@
     </dynamixel_AX12_fixed>
      <gripper_finger_base parent="gripper_servo_link" name="gripper_finger_base" color="${color}">
-      <origin xyz="${-(0.065-AX12_HEIGHT)} ${-AX12_WIDTH+0.004} ${-AX12_LENGTH/2}" rpy="${M_PI/2} 0 0"/>
+      <origin xyz="${-(0.065-AX12_HEIGHT)} ${-AX12_WIDTH+0.004} 0.0" rpy="${M_PI/2} 0 0"/>
     </gripper_finger_base>
      <!-- Finger 1 -->

File: turtlebot_arm_description/urdf/turtlebot_arm.urdf.xacro (robot description, xacro)
@@ -16,11 +16,11 @@
     <xacro:include filename="$(find turtlebot_arm_description)/urdf/turtlebot_arm.xacro"/>
     <!-- As we don't have here a turtlebot base, add a base_link link as its location reference -->
-    <link name="base_link"/>
+<!--    <link name="base_link"/> -->
     <!-- Turtlebot arm macro -->
-    <turtlebot_arm parent="base_link" color="White" gripper_color="Green"
-                    pincher_gripper="false" turtlebot_gripper="true">
+  <!--  <turtlebot_arm parent="base_link" color="White" gripper_color="Green"
+                    pincher_gripper="false" turtlebot_gripper="true">         -->
       <!-- Place the "floating" arm at the location it should be if mounted on a turtlebot,
            as pick and place and other demos assume this location -->
-      <origin xyz="0.1 0.03 0.435"/>
-    </turtlebot_arm>
+<!--      <origin xyz="0.1 0.03 0.435"/>
+    </turtlebot_arm> -->
 </robot>
